Commit message: ultimos cambios

File: urdf/bluerov.urdf.xacro (robot description, xacro)
@@ -224,3 +224,14 @@
   </xacro:macro>
   <xacro:ros2_control_sensor_system/>
+  <ros2_control name="${robot_namespace}_actuators" type="system">
+    <hardware>
+      <plugin>sura_hardware_interface/ActuatorsSystem</plugin>
+      <param name="environment">$(arg environment)</param>
+    </hardware>
+    <joint name="${robot_prefix}bluerov_lights">
+      <command_interface name="pwm_us"/>
+      <state_interface name="pwm_us"/>
+      <param name="channel">12</param>
+    </joint>
+  </ros2_control>
 </robot>

Commit message: integracion general

File: urdf/bluerov.urdf.xacro (robot description, xacro)
@@ -1,236 +1,321 @@
 <?xml version="1.0"?>
-<robot name="bluerov" xmlns:xacro="http://www.ros.org/wiki/xacro">
-  <xacro:arg name="robot_namespace" default="bluerov"/>
+<robot xmlns:xacro="http://www.ros.org/wiki/xacro" name="bluerov" family="underwater">
+  <xacro:arg name="robot_name" default="bluerov"/>
   <xacro:arg name="environment" default="real"/>
-  <xacro:arg name="lookup_csv" default="config/t200_lookup.csv"/>
-  <xacro:arg name="stonefish_topic" default="/bluerov/controller/thruster_setpoints_sim"/>
-  <xacro:arg name="pwm_channels" default="0,1,2,3,4,5,6,7"/>
-  <xacro:arg name="pressure_offset_pa" default="0.0"/>
-  <xacro:property name="robot_namespace" value="$(arg robot_namespace)"/>
-  <xacro:property name="robot_prefix" value="${robot_namespace}/"/>
-  <xacro:macro name="thruster_mount" params="link_name joint_name xyz rpy">
-    <link name="${robot_prefix}${link_name}"/>
-    <joint name="${robot_prefix}${joint_name}" type="fixed">
-      <parent link="${robot_prefix}base_link"/>
-      <child link="${robot_prefix}${link_name}"/>
-      <origin xyz="${xyz}" rpy="${rpy}"/>
-    </joint>
-  </xacro:macro>
-  <xacro:macro name="sensor_mount" params="link_name joint_name xyz rpy">
-    <link name="${link_name}"/>
-    <joint name="${joint_name}" type="fixed">
-      <parent link="${robot_prefix}base_link"/>
-      <child link="${link_name}"/>
-      <origin xyz="${xyz}" rpy="${rpy}"/>
-    </joint>
-  </xacro:macro>
-  <xacro:macro name="ros2_control_thruster_joint" params="joint_name inverted">
-    <joint name="${robot_prefix}${joint_name}">
-      <command_interface name="effort"/>
-      <state_interface name="effort"/>
-      <param name="inverted">${inverted}</param>
-    </joint>
-  </xacro:macro>
-  <link name="${robot_prefix}base_link">
+  <!-- TF -->
+  <link name="$(arg robot_name)/base_link" tf_type="base">
     <visual>
       <geometry>
         <mesh
-          filename="package://bluerov_description/urdf/bluerov/meshes/bluerov2_heavy/bluerov2_centrado.dae"
+          filename="package://bluerov_description/urdf/meshes/bluerov2_heavy/bluerov2_centrado.dae"
           scale="0.025 0.025 0.025"/>
       </geometry>
-      <origin rpy="3.1416 0 0" xyz="0 0 0"/>
+      <origin xyz="0 0 0" rpy="3.1416 0 0"/>
     </visual>
   </link>
-  <xacro:sensor_mount
-    link_name="${robot_prefix}imu_link"
-    joint_name="${robot_prefix}imu_joint"
-    xyz="0.05 0.0 -0.05"
-    rpy="-1.57 0 0"/>
-  <xacro:sensor_mount
-    link_name="${robot_prefix}dvl_link"
-    joint_name="${robot_prefix}dvl_joint"
-    xyz="0.0 -0.23 -0.05"
-    rpy="0.0 0.0 0.0"/>
-  <!-- camera down -->
-  <link name="${robot_prefix}camera_down/camera"/>
-  <joint name="${robot_prefix}camera_down_joint" type="fixed">
-    <parent link="${robot_prefix}base_link"/>
-    <child link="${robot_prefix}camera_down/camera"/>
+  <!-- Sensors -->
+  <link name="$(arg robot_name)/imu_link" tf_type="sensor"/>
+  <joint name="$(arg robot_name)/imu_joint" type="fixed">
+    <parent link="$(arg robot_name)/base_link"/>
+    <child link="$(arg robot_name)/imu_link"/>
+    <origin xyz="0.05 0.0 -0.05" rpy="-1.57 0 0"/>
+  </joint>
+  <link name="$(arg robot_name)/dvl_link" tf_type="sensor"/>
+  <joint name="$(arg robot_name)/dvl_joint" type="fixed">
+    <parent link="$(arg robot_name)/base_link"/>
+    <child link="$(arg robot_name)/dvl_link"/>
+    <origin xyz="0.0 -0.23 -0.05" rpy="0 0 0"/>
+  </joint>
+  <link name="$(arg robot_name)/pressure_link" tf_type="sensor"/>
+  <joint name="$(arg robot_name)/pressure_joint" type="fixed">
+    <parent link="$(arg robot_name)/base_link"/>
+    <child link="$(arg robot_name)/pressure_link"/>
+    <origin xyz="0 0 0" rpy="0 0 0"/>
+  </joint>
+  <link name="$(arg robot_name)/camera_down" tf_type="sensor"/>
+  <joint name="$(arg robot_name)/camera_down_joint" type="fixed">
+    <parent link="$(arg robot_name)/base_link"/>
+    <child link="$(arg robot_name)/camera_down"/>
     <origin xyz="0.006 0.13 0.143" rpy="0 0 0.0"/>
   </joint>
-  <link name="${robot_prefix}camera_down/optical_frame"/>
-  <joint name="${robot_prefix}camera_down_optical_frame_joint" type="fixed">
-    <parent link="${robot_prefix}camera_down/camera"/>
-    <child link="${robot_prefix}camera_down/optical_frame"/>
+  <link name="$(arg robot_name)/camera_down/optical_frame" tf_type="sensor"/>
+  <joint name="$(arg robot_name)/camera_down_optical_frame_joint" type="fixed">
+    <parent link="$(arg robot_name)/camera_down"/>
+    <child link="$(arg robot_name)/camera_down/optical_frame"/>
     <origin xyz="0.0 0.0 0.0" rpy="0.0 0.0 1.57"/>
   </joint>
-  <!-- camera front -->
-  <link name="${robot_prefix}camera_front"/>
-  <joint name="${robot_prefix}camera_front_joint" type="fixed">
-    <parent link="${robot_prefix}base_link"/>
-    <child link="${robot_prefix}camera_front"/>
+  <link name="$(arg robot_name)/camera_front" tf_type="sensor"/>
+  <joint name="$(arg robot_name)/camera_front_joint" type="fixed">
+    <parent link="$(arg robot_name)/base_link"/>
+    <child link="$(arg robot_name)/camera_front"/>
     <origin xyz="0.17 -0.005 -0.035" rpy="0.0 0.0 0.0"/>
   </joint>
-  <link name="${robot_prefix}camera_front/optical_frame"/>
-  <joint name="${robot_prefix}camera_front_optical_frame_joint" type="fixed">
-    <parent link="${robot_prefix}camera_front"/>
-    <child link="${robot_prefix}camera_front/optical_frame"/>
+  <link name="$(arg robot_name)/camera_front/optical_frame" tf_type="sensor"/>
+  <joint name="$(arg robot_name)/camera_front_optical_frame_joint" type="fixed">
+    <parent link="$(arg robot_name)/camera_front"/>
+    <child link="$(arg robot_name)/camera_front/optical_frame"/>
     <origin xyz="0.0 0.0 0.0" rpy="-1.57 3.14 -1.57"/>
   </joint>
-  <!-- camera right -->
-  <link name="${robot_prefix}camera_right"/>
-  <joint name="${robot_prefix}camera_right_joint" type="fixed">
-    <parent link="${robot_prefix}base_link"/>
-    <child link="${robot_prefix}camera_right"/>
+  <link name="$(arg robot_name)/camera_right" tf_type="sensor"/>
+  <joint name="$(arg robot_name)/camera_right_joint" type="fixed">
+    <parent link="$(arg robot_name)/base_link"/>
+    <child link="$(arg robot_name)/camera_right"/>
     <origin xyz="0.14 0.007 -0.1" rpy="0.0 0.0 0.0"/>
   </joint>
-  <link name="${robot_prefix}camera_right/optical_frame"/>
-  <joint name="${robot_prefix}camera_right_optical_frame_joint" type="fixed">
-    <parent link="${robot_prefix}camera_right"/>
-    <child link="${robot_prefix}camera_right/optical_frame"/>
+  <link name="$(arg robot_name)/camera_right/optical_frame" tf_type="sensor"/>
+  <joint name="$(arg robot_name)/camera_right_optical_frame_joint" type="fixed">
+    <parent link="$(arg robot_name)/camera_right"/>
+    <child link="$(arg robot_name)/camera_right/optical_frame"/>
     <origin xyz="0.0 0.0 0.0" rpy="-1.57 3.14 -1.57"/>
   </joint>
-  <!-- camera left -->
-  <link name="${robot_prefix}camera_left"/>
-  <joint name="${robot_prefix}camera_left_joint" type="fixed">
-    <parent link="${robot_prefix}base_link"/>
-    <child link="${robot_prefix}camera_left"/>
+  <link name="$(arg robot_name)/camera_left" tf_type="sensor"/>
+  <joint name="$(arg robot_name)/camera_left_joint" type="fixed">
+    <parent link="$(arg robot_name)/base_link"/>
+    <child link="$(arg robot_name)/camera_left"/>
     <origin xyz="0.14 -0.06 -0.1" rpy="0.0 0.0 0.0"/>
   </joint>
-  <link name="${robot_prefix}camera_left/optical_frame"/>
-  <joint name="${robot_prefix}camera_left_optical_frame_joint" type="fixed">
-    <parent link="${robot_prefix}camera_left"/>
-    <child link="${robot_prefix}camera_left/optical_frame"/>
+  <link name="$(arg robot_name)/camera_left/optical_frame" tf_type="sensor"/>
+  <joint name="$(arg robot_name)/camera_left_optical_frame_joint" type="fixed">
+    <parent link="$(arg robot_name)/camera_left"/>
+    <child link="$(arg robot_name)/camera_left/optical_frame"/>
     <origin xyz="0.0 0.0 0.0" rpy="-1.57 3.14 -1.57"/>
   </joint>
-  <xacro:thruster_mount
-    link_name="Thruster_R_FORWARD_FRONT"
-    joint_name="Thruster_R_FORWARD_FRONT"
-    xyz="0.145737 0.091717 0.04783"
-    rpy="0.0 0.0 -0.7853"/>
-  <xacro:thruster_mount
-    link_name="Thruster_L_FORWARD_FRONT"
-    joint_name="Thruster_L_FORWARD_FRONT"
-    xyz="0.145737 -0.09814 0.04783"
-    rpy="0.0 0.0 0.7853"/>
-  <xacro:thruster_mount
-    link_name="Thruster_R_FORWARD_REAR"
-    joint_name="Thruster_R_FORWARD_REAR"
-    xyz="-0.145419 0.091717 0.04783"
-    rpy="0.0 0.0 -2.35619"/>
-  <xacro:thruster_mount
-    link_name="Thruster_L_FORWARD_REAR"
-    joint_name="Thruster_L_FORWARD_REAR"
-    xyz="-0.145419 -0.09814 0.04783"
-    rpy="0.0 0.0 2.35619"/>
-  <xacro:thruster_mount
-    link_name="Thruster_R_UP_FRONT"
-    joint_name="Thruster_R_UP_FRONT"
-    xyz="0.124709 0.209 -0.013231"
-    rpy="1.57 1.57 0.0"/>
-  <xacro:thruster_mount
-    link_name="Thruster_L_UP_FRONT"
-    joint_name="Thruster_L_UP_FRONT"
-    xyz="0.124709 -0.220356 -0.013231"
-    rpy="1.57 1.57 0.0"/>
-  <xacro:thruster_mount
-    link_name="Thruster_R_UP_REAR"
-    joint_name="Thruster_R_UP_REAR"
-    xyz="-0.112476 0.209 -0.013231"
-    rpy="1.57 1.57 0.0"/>
-  <xacro:thruster_mount
-    link_name="Thruster_L_UP_REAR"
-    joint_name="Thruster_L_UP_REAR"
-    xyz="-0.112476 -0.220356 -0.013231"
-    rpy="1.57 1.57 0.0"/>
-  <ros2_control name="${robot_namespace}_thrusters" type="system">
+  <!-- Thrusters -->
+  <link name="$(arg robot_name)/Thruster_R_FORWARD_FRONT" tf_type="thruster"/>
+  <joint name="$(arg robot_name)/Thruster_R_FORWARD_FRONT" type="fixed">
+    <parent link="$(arg robot_name)/base_link"/>
+    <child link="$(arg robot_name)/Thruster_R_FORWARD_FRONT"/>
+    <origin xyz="0.145737 0.091717 0.04783" rpy="0.0 0.0 -0.7853"/>
+  </joint>
+  <link name="$(arg robot_name)/Thruster_L_FORWARD_FRONT" tf_type="thruster"/>
+  <joint name="$(arg robot_name)/Thruster_L_FORWARD_FRONT" type="fixed">
+    <parent link="$(arg robot_name)/base_link"/>
+    <child link="$(arg robot_name)/Thruster_L_FORWARD_FRONT"/>
+    <origin xyz="0.145737 -0.09814 0.04783" rpy="0.0 0.0 0.7853"/>
+  </joint>
+  <link name="$(arg robot_name)/Thruster_R_FORWARD_REAR" tf_type="thruster"/>
+  <joint name="$(arg robot_name)/Thruster_R_FORWARD_REAR" type="fixed">
+    <parent link="$(arg robot_name)/base_link"/>
+    <child link="$(arg robot_name)/Thruster_R_FORWARD_REAR"/>
+    <origin xyz="-0.145419 0.091717 0.04783" rpy="0.0 0.0 -2.35619"/>
+  </joint>
+  <link name="$(arg robot_name)/Thruster_L_FORWARD_REAR" tf_type="thruster"/>
+  <joint name="$(arg robot_name)/Thruster_L_FORWARD_REAR" type="fixed">
+    <parent link="$(arg robot_name)/base_link"/>
+    <child link="$(arg robot_name)/Thruster_L_FORWARD_REAR"/>
+    <origin xyz="-0.145419 -0.09814 0.04783" rpy="0.0 0.0 2.35619"/>
+  </joint>
+  <link name="$(arg robot_name)/Thruster_R_UP_FRONT" tf_type="thruster"/>
+  <joint name="$(arg robot_name)/Thruster_R_UP_FRONT" type="fixed">
+    <parent link="$(arg robot_name)/base_link"/>
+    <child link="$(arg robot_name)/Thruster_R_UP_FRONT"/>
+    <origin xyz="0.124709 0.209 -0.013231" rpy="1.57 1.57 0.0"/>
+  </joint>
+  <link name="$(arg robot_name)/Thruster_L_UP_FRONT" tf_type="thruster"/>
+  <joint name="$(arg robot_name)/Thruster_L_UP_FRONT" type="fixed">
+    <parent link="$(arg robot_name)/base_link"/>
+    <child link="$(arg robot_name)/Thruster_L_UP_FRONT"/>
+    <origin xyz="0.124709 -0.220356 -0.013231" rpy="1.57 1.57 0.0"/>
+  </joint>
+  <link name="$(arg robot_name)/Thruster_R_UP_REAR" tf_type="thruster"/>
+  <joint name="$(arg robot_name)/Thruster_R_UP_REAR" type="fixed">
+    <parent link="$(arg robot_name)/base_link"/>
+    <child link="$(arg robot_name)/Thruster_R_UP_REAR"/>
+    <origin xyz="-0.112476 0.209 -0.013231" rpy="1.57 1.57 0.0"/>
+  </joint>
+  <link name="$(arg robot_name)/Thruster_L_UP_REAR" tf_type="thruster"/>
+  <joint name="$(arg robot_name)/Thruster_L_UP_REAR" type="fixed">
+    <parent link="$(arg robot_name)/base_link"/>
+    <child link="$(arg robot_name)/Thruster_L_UP_REAR"/>
+    <origin xyz="-0.112476 -0.220356 -0.013231" rpy="1.57 1.57 0.0"/>
+  </joint>
+  <!-- Actuators -->
+  <link name="$(arg robot_name)/lights_link" tf_type="actuator"/>
+  <joint name="$(arg robot_name)/lights_joint" type="fixed">
+    <parent link="$(arg robot_name)/base_link"/>
+    <child link="$(arg robot_name)/lights_link"/>
+    <origin xyz="0 0 0" rpy="0 0 0"/>
+  </joint>
+  <!-- ROS2 CONTROL -->
+  <ros2_control name="$(arg robot_name)_thrusters" type="system">
     <hardware>
       <plugin>sura_hardware_interface/ThrustersSystem</plugin>
       <param name="environment">$(arg environment)</param>
-      <param name="lookup_csv">$(arg lookup_csv)</param>
-      <param name="stonefish_topic">$(arg stonefish_topic)</param>
-      <param name="pwm_channels">$(arg pwm_channels)</param>
     </hardware>
-    <xacro:ros2_control_thruster_joint joint_name="Thruster_R_FORWARD_FRONT" inverted="false"/>
-    <xacro:ros2_control_thruster_joint joint_name="Thruster_L_FORWARD_FRONT" inverted="false"/>
-    <xacro:ros2_control_thruster_joint joint_name="Thruster_R_FORWARD_REAR" inverted="true"/>
-    <xacro:ros2_control_thruster_joint joint_name="Thruster_L_FORWARD_REAR" inverted="true"/>
-    <xacro:ros2_control_thruster_joint joint_name="Thruster_R_UP_FRONT" inverted="false"/>
-    <xacro:ros2_control_thruster_joint joint_name="Thruster_L_UP_FRONT" inverted="true"/>
-    <xacro:ros2_control_thruster_joint joint_name="Thruster_R_UP_REAR" inverted="true"/>
-    <xacro:ros2_control_thruster_joint joint_name="Thruster_L_UP_REAR" inverted="false"/>
+    <joint name="$(arg robot_name)/Thruster_R_FORWARD_FRONT">
+      <command_interface name="effort"/>
+      <state_interface name="effort"/>
+      <param name="lookup_csv">config/t200_lookup.csv</param>
+      <param name="stonefish_topic">/$(arg robot_name)/controller/thruster_setpoints_sim</param>
+      <param name="inverted">false</param>
+      <param name="pwm_offset">0.0</param>
+      <param name="channel">0</param>
+    </joint>
+    <joint name="$(arg robot_name)/Thruster_L_FORWARD_FRONT">
+      <command_interface name="effort"/>
+      <state_interface name="effort"/>
+      <param name="lookup_csv">config/t200_lookup.csv</param>
+      <param name="stonefish_topic">/$(arg robot_name)/controller/thruster_setpoints_sim</param>
+      <param name="inverted">false</param>
+      <param name="pwm_offset">0.0</param>
+      <param name="channel">1</param>
+    </joint>
+    <joint name="$(arg robot_name)/Thruster_R_FORWARD_REAR">
+      <command_interface name="effort"/>
+      <state_interface name="effort"/>
+      <param name="lookup_csv">config/t200_lookup.csv</param>
+      <param name="stonefish_topic">/$(arg robot_name)/controller/thruster_setpoints_sim</param>
+      <param name="inverted">true</param>
+      <param name="pwm_offset">0.0</param>
+      <param name="channel">2</param>
+    </joint>
+    <joint name="$(arg robot_name)/Thruster_L_FORWARD_REAR">
+      <command_interface name="effort"/>
+      <state_interface name="effort"/>
+      <param name="lookup_csv">config/t200_lookup.csv</param>
+      <param name="stonefish_topic">/$(arg robot_name)/controller/thruster_setpoints_sim</param>
+      <param name="inverted">true</param>
+      <param name="pwm_offset">0.0</param>
+      <param name="channel">3</param>
+    </joint>
+    <joint name="$(arg robot_name)/Thruster_R_UP_FRONT">
+      <command_interface name="effort"/>
+      <state_interface name="effort"/>
+      <param name="lookup_csv">config/t200_lookup.csv</param>
+      <param name="stonefish_topic">/$(arg robot_name)/controller/thruster_setpoints_sim</param>
+      <param name="inverted">false</param>
+      <param name="pwm_offset">0.0</param>
+      <param name="channel">4</param>
+    </joint>
+    <joint name="$(arg robot_name)/Thruster_L_UP_FRONT">
+      <command_interface name="effort"/>
+      <state_interface name="effort"/>
+      <param name="lookup_csv">config/t200_lookup.csv</param>
+      <param name="stonefish_topic">/$(arg robot_name)/controller/thruster_setpoints_sim</param>
+      <param name="inverted">true</param>
+      <param name="pwm_offset">0.0</param>
+      <param name="channel">5</param>
+    </joint>
+    <joint name="$(arg robot_name)/Thruster_R_UP_REAR">
+      <command_interface name="effort"/>
+      <state_interface name="effort"/>
+      <param name="lookup_csv">config/t200_lookup.csv</param>
+      <param name="stonefish_topic">/$(arg robot_name)/controller/thruster_setpoints_sim</param>
+      <param name="inverted">true</param>
+      <param name="pwm_offset">0.0</param>
+      <param name="channel">6</param>
+    </joint>
+    <joint name="$(arg robot_name)/Thruster_L_UP_REAR">
+      <command_interface name="effort"/>
+      <state_interface name="effort"/>
+      <param name="lookup_csv">config/t200_lookup.csv</param>
+      <param name="stonefish_topic">/$(arg robot_name)/controller/thruster_setpoints_sim</param>
+      <param name="inverted">false</param>
+      <param name="pwm_offset">0.0</param>
+      <param name="channel">7</param>
+    </joint>
   </ros2_control>
-  <xacro:macro name="ros2_control_sensor_system">
-    <ros2_control name="${robot_namespace}_sensors" type="system">
-      <hardware>
-        <plugin>sura_hardware_interface/SensorsSystem</plugin>
-        <param name="environment">$(arg environment)</param>
-        <param name="robot_namespace">${robot_namespace}</param>
-        <param name="sim_imu_topic">/${robot_namespace}/stonefish/sensors/imu</param>
-        <param name="sim_magnetometer_topic">/${robot_namespace}/stonefish/sensors/magnetometer</param>
-        <param name="sim_pressure_topic">/${robot_namespace}/stonefish/sensors/pressure</param>
-        <param name="sim_dvl_topic">/${robot_namespace}/stonefish/sensors/dvl</param>
-        <param name="sim_dvl_altitude_topic">/${robot_namespace}/stonefish/sensors/dvl/altitude</param>
-        <param name="sim_gps_topic">/${robot_namespace}/stonefish/sensors/gps</param>
-        <param name="pressure_offset_pa">$(arg pressure_offset_pa)</param>
-        <param name="pressure_read_rate_hz">200.0</param>
-        <param name="dvl_read_rate_hz">20.0</param>
-        <param name="battery_read_rate_hz">1.0</param>
-        <param name="leak_read_rate_hz">1.0</param>
-      </hardware>
-      <sensor name="imu_sensor">
-        <state_interface name="orientation.x"/>
-        <state_interface name="orientation.y"/>
-        <state_interface name="orientation.z"/>
-        <state_interface name="orientation.w"/>
-        <state_interface name="angular_velocity.x"/>
-        <state_interface name="angular_velocity.y"/>
-        <state_interface name="angular_velocity.z"/>
-        <state_interface name="linear_acceleration.x"/>
-        <state_interface name="linear_acceleration.y"/>
-        <state_interface name="linear_acceleration.z"/>
-      </sensor>
-      <sensor name="magnetometer_sensor">
-        <state_interface name="magnetic_field.x"/>
-        <state_interface name="magnetic_field.y"/>
-        <state_interface name="magnetic_field.z"/>
-      </sensor>
-      <sensor name="pressure_sensor">
-        <state_interface name="fluid_pressure"/>
-      </sensor>
-      <sensor name="battery_sensor">
-        <state_interface name="voltage"/>
-        <state_interface name="current"/>
-        <state_interface name="present"/>
-      </sensor>
-      <sensor name="leak_sensor">
-        <state_interface name="leak"/>
-      </sensor>
-      <sensor name="dvl_sensor">
-        <state_interface name="linear_velocity.x"/>
-        <state_interface name="linear_velocity.y"/>
-        <state_interface name="linear_velocity.z"/>
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