Commit message: arreglos imu

File: urdf/bigblue.urdf.xacro (robot description, xacro)
@@ -19,5 +19,5 @@
     <parent link="$(arg robot_name)/base_link"/>
     <child link="$(arg robot_name)/imu_link"/>
-    <origin xyz="0.05 0.0 -0.05" rpy="-1.57 0 0"/>
+    <origin xyz="0.1043 -0.083264 -0.0547" rpy="-1.57 0 0"/>
   </joint>
   <link name="$(arg robot_name)/dvl_link" tf_type="sensor"/>
@@ -80,4 +80,10 @@
     <child link="$(arg robot_name)/camera_left/optical_frame"/>
     <origin xyz="0.0 0.0 0.0" rpy="-1.57 3.14 -1.57"/>
+  </joint>
+  <link name="zed_camera_camera_link" tf_type="fixed"/>
+  <joint name="$(arg robot_name)/zed_camera_joint" type="fixed">
+    <parent link="$(arg robot_name)/base_link"/>
+    <child link="zed_camera_camera_link"/>
+    <origin xyz="0.195659 0.1 -0.04" rpy="3.1416 0.0 0.0"/>
   </joint>
   <!-- Thrusters -->
@@ -254,5 +260,5 @@
       <state_interface name="sample_time.nanosec"/>
     </sensor>
-    <sensor name="pressure_sensor">
+    <!-- <sensor name="pressure_sensor">
       <param name="interface">sura_hardware_interface/PressureInterface</param>
       <param name="broadcaster">pressure_broadcaster</param>
@@ -265,5 +271,5 @@
       <param name="msg_type">sensor_msgs/msg/FluidPressure</param>
       <state_interface name="fluid_pressure"/>
-    </sensor>
+    </sensor> -->
     <sensor name="dvl_sensor">
       <param name="interface">sura_hardware_interface/DvlInterface</param>
